Commit message: 2

File: seokgyun_description/urdf/piot.urdf (robot description, URDF)
Before this commit: robot stella, 4 links, 3 joints
Joints:
- joint base_joint: child base_footprint -> base_link; origin xyz=0.0 0.0 ${-(wheel_radius)} rpy=0 0 0 -> xyz=0.0 0.0 ${(wheel_radius)} rpy=0 0 0; parent base_link -> base_footprint
- joint imu_joint: origin xyz=${base_length/2 -lidar_xoff } ${imu_yoff} ${base_height} rpy=0.0 0.0 0.0 -> xyz=${base_length/2 -lidar_xoff } ${-imu_yoff} ${base_height} rpy=0.0 0.0 0.0

Commit message: third

File: seokgyun_description/urdf/piot.urdf (robot description, URDF)
Before this commit: robot stella, 4 links, 3 joints
Joints:
- joint imu_joint: origin xyz=${base_length/2 -lidar_xoff } ${-imu_yoff} ${base_height} rpy=0.0 0.0 0.0 -> xyz=${base_length/2 -lidar_xoff } ${-imu_yoff} ${base_height} rpy=0.0 0.0 3.14
- joint scan_joint: origin xyz=${base_length/2 -lidar_xoff } 0.0 ${base_height} rpy=0.0 0.0 0.0 -> xyz=${base_length/2 -lidar_xoff } 0.0 ${base_height} rpy=0.0 0.0 3.14

Commit message: 8

File: seokgyun_description/urdf/piot.urdf (robot description, URDF)
Before this commit: robot stella, 4 links, 3 joints
Links:
- added link camera_link
- added link gps_link
Joints:
- added joint depth_camera_joint: type fixed, parent base_link, child camera_link, origin xyz=${base_length/2} 0.0 ${base_height} rpy=0.0 0.0 0.0
- added joint gps_joint: type fixed, parent base_link, child gps_link, origin xyz=${base_length/2 } ${imu_yoff} ${base_height} rpy=0.0 0.0 0.0
- joint imu_joint: origin xyz=${base_length/2 -lidar_xoff } ${-imu_yoff} ${base_height} rpy=0.0 0.0 3.14 -> xyz=${base_length/2 -lidar_xoff } ${-imu_yoff} ${base_height} rpy=0.0 0.0 0.0

Commit message: 07-25

File: seokgyun_description/urdf/piot.urdf (robot description, URDF)
Before this commit: robot stella, 6 links, 5 joints
Joints:
- joint scan_joint: origin xyz=${base_length/2 -lidar_xoff } 0.0 ${base_height} rpy=0.0 0.0 3.14 -> xyz=${base_length/2 -lidar_xoff } 0.0 ${base_height} rpy=0.0 0.0 0.0
